Commit message: jazzy nav2 sim done - will update readme soon

File: ros2_ws/src/scoutmini_description/urdf/scout_mini/scout_mini.xacro (robot description, xacro)
@@ -8,12 +8,12 @@
     <xacro:property name="M_PI" value="3.14159"/>
     <!-- Vehicle Geometries -->
-    <xacro:property name="base_x_size" value="0.6200000" />
-    <xacro:property name="base_y_size" value="0.585000" />
-    <xacro:property name="base_z_size" value="0.235000" />
-    <xacro:property name="wheelbase" value="0.463951"/>
-    <xacro:property name="track" value="0.416503"/>
-    <xacro:property name="wheel_vertical_offset" value="-0.100998" />
-    <xacro:property name="wheel_length" value="0.8e-01" />
-    <xacro:property name="wheel_radius" value="1.600e-01" />
+    <xacro:property name="base_x_size" value="0.595000" />
+    <xacro:property name="base_y_size" value="0.395000" />
+    <xacro:property name="base_z_size" value="0.130000" />
+    <xacro:property name="wheelbase" value="0.452"/>
+    <xacro:property name="track" value="0.49"/>
+    <xacro:property name="wheel_vertical_offset" value="-0.0905" />
+    <xacro:property name="wheel_length" value="0.8520e-01" />
+    <xacro:property name="wheel_radius" value="0.8750e-01" />
     <!-- Nav2 uses base_footprint as the planar ground frame. -->
     <link name="base_footprint"/>
@@ -45,7 +45,7 @@
     <link name="inertial_link">
         <inertial>
-            <mass value="60" />
+            <mass value="23" />
             <origin xyz="0.0 0.0 0.0" />
-            <inertia ixx="2.288641" ixy="0" ixz="0" iyy="5.103976" iyz="0" izz="3.431465" />
+            <inertia ixx="0.2594" ixy="0" ixz="0" iyy="0.5567" iyz="0" izz="0.7648" />
         </inertial>
     </link>

File: ros2_ws/src/scoutmini_description/urdf/scout_mini_wheel.xacro (robot description, xacro)
@@ -6,5 +6,5 @@
                 <mass value="3" />
                 <origin xyz="0 0 0" />
-                <inertia ixx="0.7171" ixy="0" ixz="0" iyy="0.7171" iyz="0" izz="0.1361" />
+                <inertia ixx="0.00756" ixy="0" ixz="0" iyy="0.00756" iyz="0" izz="0.01148" />
             </inertial>
             <visual>
@@ -19,6 +19,5 @@
                 rpy="0 0 0" />
               <geometry>
-                <mesh
-                  filename="file://$(find scoutmini_description)/meshes/wheel.dae" />
+                <cylinder radius="${wheel_radius}" length="${wheel_length}"/>
               </geometry>
             </collision>
@@ -31,8 +30,8 @@
         </joint>
         <gazebo reference="${wheel_prefix}_wheel_link">
-            <mu1 value="1.0"/>
-            <mu2 value="0.08"/>
+            <mu1 value="1.5"/>
+            <mu2 value="0.8"/>
             <slip1 value="0.0"/>
-            <slip2 value="0.4"/>
+            <slip2 value="0.0"/>
             <kp value="500000.0"/>
             <kd value="20.0"/>

Commit message: fixed PR comments; added scoutmini_sim

File: ros2_ws/src/scoutmini_description/urdf/scout_mini/scout_mini.xacro (robot description, xacro)
@@ -3,6 +3,7 @@
     <xacro:arg name="robot_namespace" default="/" />
     <xacro:arg name="urdf_extras" default="empty.urdf" />
-    <xacro:include filename="$(find scoutmini_description)/urdf/scout_mini_wheel.xacro" />
-    <xacro:include filename="$(find scoutmini_description)/urdf/sensors.xacro" />
+    <xacro:arg name="sim" default="false" />
+    <xacro:include filename="../scout_mini_wheel.xacro" />
+    <xacro:include filename="../sensors.xacro" />
     <!-- Variables -->
     <xacro:property name="M_PI" value="3.14159"/>
@@ -47,5 +48,5 @@
             <mass value="23" />
             <origin xyz="0.0 0.0 0.0" />
-            <inertia ixx="0.2594" ixy="0" ixz="0" iyy="0.5567" iyz="0" izz="0.7648" />
+            <inertia ixx="2.288641" ixy="0" ixz="0" iyy="5.103976" iyz="0" izz="3.431465" />
         </inertial>
     </link>
@@ -82,5 +83,5 @@
         <child link="rear_mount" />
     </joint>
-    <xacro:sensor_macro parent_link="base_link">
+    <xacro:sensor_macro parent_link="base_link" sim="$(arg sim)">
         <origin xyz="0.01 0 0.07" rpy="0 0 0"/>
     </xacro:sensor_macro>
@@ -88,5 +89,5 @@
     <xacro:include filename="$(arg urdf_extras)" />
     <!-- Gazebo definitions  -->
-    <xacro:include filename="$(find scoutmini_description)/urdf/scout_mini/scout_mini.gazebo" />
+    <xacro:include filename="scout_mini.gazebo" />
     <ros2_control name="ScoutMiniSystem" type="system">
         <hardware>

File: ros2_ws/src/scoutmini_description/urdf/scout_mini_wheel.xacro (robot description, xacro)
@@ -1,2 +1,8 @@
+<!--
+  Adapted from:
+  https://github.com/agilexrobotics/scout_ros/scout_description/urdf/scout_mini_wheel.xacro
+  Original work Copyright (c) AgileX Robotics.
+  Licensed under the BSD License.
+-->
 <?xml version="1.0"?>
 <robot xmlns:xacro="http://ros.org/wiki/xacro" name="scout_wheel">

File: ros2_ws/src/scoutmini_description/urdf/sensors.xacro (robot description, xacro)
@@ -1,6 +1,14 @@
 <?xml version="1.0"?>
 <robot xmlns:xacro="http://ros.org/wiki/xacro">
-  <xacro:macro name="sensor_macro" params="parent_link:=base_link *origin">
+  <xacro:macro name="sensor_macro" params="parent_link:=base_link sim:=false *origin">
     <xacro:arg name="camera_name"   default="zed2" />
+    <xacro:arg name="camera_model"  default="zed2" />
+    <xacro:unless value="${sim}">
+      <!-- Real ZED camera for the physical robot. -->
+      <xacro:include filename="$(find zed_wrapper)/urdf/zed_macro.urdf.xacro" />
+      <xacro:zed_camera name="$(arg camera_name)" model="$(arg camera_model)" custom_baseline="0.0" enable_gnss="false">
+        <origin xyz="0 0 0" rpy="0 0 0"/>
+      </xacro:zed_camera>
+    </xacro:unless>
     <!-- Sensor Link -->
     <link name="sensor_link">
@@ -124,25 +132,27 @@
       <origin xyz="-0.16 0 0.0" rpy="0 0 0"/>  <!-- Adjust position -->
     </joint>
-    <!-- Simulated ZED replacement: a normal forward-facing RGB camera. -->
-    <link name="$(arg camera_name)_camera_link">
-      <visual>
-        <geometry>
-          <box size="0.09 0.16 0.05"/>
-        </geometry>
-        <material name="sim_zed_camera_material">
-          <color rgba="0.05 0.05 0.05 1.0"/>
-        </material>
-      </visual>
-      <collision>
-        <geometry>
-          <box size="0.09 0.16 0.05"/>
-        </geometry>
-      </collision>
-      <inertial>
-        <mass value="0.15"/>
-        <origin xyz="0 0 0" rpy="0 0 0"/>
-        <inertia ixx="0.0001" ixy="0" ixz="0" iyy="0.0001" iyz="0" izz="0.0001"/>
-      </inertial>
-    </link>
+    <xacro:if value="${sim}">
+      <!-- Simulated ZED replacement: a normal forward-facing RGB camera. -->
+      <link name="$(arg camera_name)_camera_link">
+        <visual>
+          <geometry>
+            <box size="0.09 0.16 0.05"/>
+          </geometry>
+          <material name="sim_zed_camera_material">
+            <color rgba="0.05 0.05 0.05 1.0"/>
+          </material>
+        </visual>
+        <collision>
+          <geometry>
+            <box size="0.09 0.16 0.05"/>
+          </geometry>
+        </collision>
+        <inertial>
+          <mass value="0.15"/>
+          <origin xyz="0 0 0" rpy="0 0 0"/>
+          <inertia ixx="0.0001" ixy="0" ixz="0" iyy="0.0001" iyz="0" izz="0.0001"/>
+        </inertial>
+      </link>
+    </xacro:if>
     <joint name="$(arg camera_name)_joint" type="fixed">
       <parent link="sensor_to_cams_link"/>
@@ -150,36 +160,38 @@
       <origin xyz="0.055 0.0 0.415" rpy="0 0 0"/>
     </joint>
-    <link name="$(arg camera_name)_camera_optical_frame"/>
-    <joint name="$(arg camera_name)_camera_optical_joint" type="fixed">
-      <parent link="$(arg camera_name)_camera_link"/>
-      <child link="$(arg camera_name)_camera_optical_frame"/>
-      <origin xyz="0.045 0 0" rpy="-1.57079632679 0 -1.57079632679"/>
-    </joint>
-    <gazebo reference="$(arg camera_name)_camera_optical_frame">
-      <sensor name="$(arg camera_name)_rgb_camera" type="camera">
-        <always_on>true</always_on>
-        <update_rate>30</update_rate>
-        <visualize>true</visualize>
-        <topic>/$(arg camera_name)/zed_node/rgb/color/rect/image</topic>
-        <gz_frame_id>$(arg camera_name)_camera_optical_frame</gz_frame_id>
-        <camera>
-          <horizontal_fov>1.3962634</horizontal_fov>
-          <image>
-            <width>1280</width>
-            <height>720</height>
-            <format>R8G8B8</format>
-          </image>
-          <clip>
-            <near>0.05</near>
-            <far>50.0</far>
-          </clip>
-          <noise>
-            <type>gaussian</type>
-            <mean>0.0</mean>
-            <stddev>0.005</stddev>
-          </noise>
-        </camera>
-      </sensor>
-    </gazebo>
+    <xacro:if value="${sim}">
+      <link name="$(arg camera_name)_camera_optical_frame"/>
+      <joint name="$(arg camera_name)_camera_optical_joint" type="fixed">
+        <parent link="$(arg camera_name)_camera_link"/>
+        <child link="$(arg camera_name)_camera_optical_frame"/>
+        <origin xyz="0.045 0 0" rpy="-1.57079632679 0 -1.57079632679"/>
+      </joint>
+      <gazebo reference="$(arg camera_name)_camera_optical_frame">
+        <sensor name="$(arg camera_name)_rgb_camera" type="camera">
+          <always_on>true</always_on>
+          <update_rate>30</update_rate>
+          <visualize>true</visualize>
+          <topic>/$(arg camera_name)/zed_node/rgb/color/rect/image</topic>
+          <gz_frame_id>$(arg camera_name)_camera_optical_frame</gz_frame_id>
+          <camera>
+            <horizontal_fov>1.3962634</horizontal_fov>
+            <image>
+              <width>1280</width>
+              <height>720</height>
+              <format>R8G8B8</format>
+            </image>
+            <clip>
+              <near>0.05</near>
+              <far>50.0</far>
+            </clip>
+            <noise>
+              <type>gaussian</type>
+              <mean>0.0</mean>
+              <stddev>0.005</stddev>
+            </noise>
+          </camera>
+        </sensor>
+      </gazebo>
+    </xacro:if>
     <!-- Simulated Insta360 replacement: a normal RGB camera publishing on the equirectangular image topic. -->
     <link name="insta360_camera_link">

Commit message: final changes

File: ros2_ws/src/scoutmini_description/urdf/scout_mini/scout_mini.xacro (robot description, xacro)
@@ -4,6 +4,7 @@
     <xacro:arg name="urdf_extras" default="empty.urdf" />
     <xacro:arg name="sim" default="false" />
-    <xacro:include filename="../scout_mini_wheel.xacro" />
-    <xacro:include filename="../sensors.xacro" />
+    <xacro:include filename="$(find scoutmini_description)/urdf/scout_mini_wheel.xacro" />
+    <!-- Sensors -->
+    <xacro:include filename="$(find scoutmini_description)/urdf/sensors.xacro" />
     <!-- Variables -->
     <xacro:property name="M_PI" value="3.14159"/>
@@ -71,16 +72,4 @@
         <origin xyz="${-wheelbase/2} ${-track/2} ${wheel_vertical_offset}" rpy="1.57 0 0" />
     </xacro:scout_mini_wheel>
-    <link name="front_mount" />
-    <joint name="front_mount_joint" type="fixed">
-        <origin xyz="0.175 0 0.068999" rpy="0 0 0" />
-        <parent link="base_link" />
-        <child link="front_mount" />
-    </joint>
-    <link name="rear_mount" />
-    <joint name="rear_mount_joint" type="fixed">
-        <origin xyz="-0.175 0 0.068999" rpy="0 0 0" />
-        <parent link="base_link" />
-        <child link="rear_mount" />
-    </joint>
     <xacro:sensor_macro parent_link="base_link" sim="$(arg sim)">
         <origin xyz="0.01 0 0.07" rpy="0 0 0"/>
