Commit message: Created Gazebo Simulation for Scout Mini (with Nav2 capabilities) (#3)
* complete urdf/xacro for scout mini

* gazebo linear movement

* changed zed-ros2-wrapper back to original

* gazebo with sensors: zed and insta360 replaced with rgb cameras

* Initial nav2 (map stuck on fuse3rd)

* jazzy nav2 sim done - will update readme soon

* humble working

* better robot rotational motion

* better nav2 params, added sim instructions readme in scoutmini_nav2

* added fuse_3rd world sdf; important nav2 changes

* fixed PR comments; added scoutmini_sim

* final changes

---------

Co-authored-by: Nhat Le <nhatleminh1997@gmail.com>

File: ros2_ws/src/scoutmini_description/urdf/scout_mini/scout_mini.xacro (robot description, xacro)
@@ -1,7 +1,8 @@
 <?xml version="1.0"?>
-<robot name="scout_mini"
-    xmlns:xacro="http://ros.org/wiki/xacro">
+<robot name="scout_mini" xmlns:xacro="http://ros.org/wiki/xacro">
     <xacro:arg name="robot_namespace" default="/" />
-    <xacro:include filename="$(find scout_description)/urdf/scout_mini/scout_mini_wheel.xacro" />
+    <xacro:arg name="urdf_extras" default="empty.urdf" />
+    <xacro:arg name="sim" default="false" />
+    <xacro:include filename="$(find scoutmini_description)/urdf/scout_mini_wheel.xacro" />
     <!-- Sensors -->
     <xacro:include filename="$(find scoutmini_description)/urdf/sensors.xacro" />
@@ -10,36 +11,41 @@
     <!-- Vehicle Geometries -->
     <xacro:property name="base_x_size" value="0.595000" />
-    <!-- <xacro:property name="base_y_size" value="0.335000" /> -->
     <xacro:property name="base_y_size" value="0.395000" />
     <xacro:property name="base_z_size" value="0.130000" />
-    <xacro:property name="wheelbase" value="0.452" />
-    <xacro:property name="track" value="0.49" />
+    <xacro:property name="wheelbase" value="0.452"/>
+    <xacro:property name="track" value="0.49"/>
     <xacro:property name="wheel_vertical_offset" value="-0.0905" />
     <xacro:property name="wheel_length" value="0.8520e-01" />
     <xacro:property name="wheel_radius" value="0.8750e-01" />
+    <!-- Nav2 uses base_footprint as the planar ground frame. -->
+    <link name="base_footprint"/>
+    <joint name="base_footprint_joint" type="fixed">
+        <origin xyz="0 0 ${wheel_radius - wheel_vertical_offset}" rpy="0 0 0" />
+        <parent link="base_footprint" />
+        <child link="base_link" />
+    </joint>
     <!-- Base link -->
     <link name="base_link">
         <visual>
-            <origin xyz="0 0 0" rpy="0 0 0" />
+            <origin
+                    xyz="0 0 0"
+                    rpy="1.5707 0 -1.5707" />
             <geometry>
-                <mesh filename="package://scout_description/meshes/scout_mini/mini_base_link.dae" />
+                <mesh filename="file://$(find scoutmini_description)/meshes/scout_mini_base_link.dae" />
             </geometry>
         </visual>
         <collision>
-            <origin xyz="0 0 0.008" rpy="0 0 0" />
-            <geometry>
-                <box size="${base_x_size} ${base_y_size} ${base_z_size}"/>
-            </geometry>
+            <origin
+                    xyz="0 0 0"
+                    rpy="1.5707 0 -1.5707" />
+          <geometry>
+            <mesh
+              filename="file://$(find scoutmini_description)/meshes/scout_mini_base_link.dae" />
+          </geometry>
         </collision>
     </link>
-    <link name="base_footprint"/>
-    <joint name="base_footprint_joint" type="fixed">
-        <origin xyz="0 0 ${wheel_vertical_offset - wheel_radius}" rpy="0 0 0" />
-        <parent link="base_link" />
-        <child link="base_footprint" />
-    </joint>
     <link name="inertial_link">
         <inertial>
-            <mass value="18" />
+            <mass value="23" />
             <origin xyz="0.0 0.0 0.0" />
             <inertia ixx="2.288641" ixy="0" ixz="0" iyy="5.103976" iyz="0" izz="3.431465" />
@@ -55,17 +61,46 @@
     <!-- motor 1 and 2 (left side) are mechanically installed in a reversed direction -->
     <xacro:scout_mini_wheel wheel_prefix="front_right">
-        <origin xyz="${wheelbase/2} ${-track/2} ${wheel_vertical_offset}" rpy="3.14 0 0" />
+        <origin xyz="${wheelbase/2} ${-track/2} ${wheel_vertical_offset}" rpy="1.57 0 0" />
     </xacro:scout_mini_wheel>
-    <xacro:scout_mini_wheel wheel_prefix="front_left">
-        <origin xyz="${wheelbase/2} ${track/2} ${wheel_vertical_offset}" rpy="0 0 0" />
+    <xacro:scout_mini_wheel wheel_prefix="front_left" wheel_axis="0 0 1">
+        <origin xyz="${wheelbase/2} ${track/2} ${wheel_vertical_offset}" rpy="-1.57 0 0" />
     </xacro:scout_mini_wheel>
-    <xacro:scout_mini_wheel wheel_prefix="rear_left">
-        <origin xyz="${-wheelbase/2} ${track/2} ${wheel_vertical_offset}" rpy="0 0 0" />
+    <xacro:scout_mini_wheel wheel_prefix="rear_left" wheel_axis="0 0 1">
+        <origin xyz="${-wheelbase/2} ${track/2} ${wheel_vertical_offset}" rpy="-1.57 0 0" />
     </xacro:scout_mini_wheel>
     <xacro:scout_mini_wheel wheel_prefix="rear_right">
-        <origin xyz="${-wheelbase/2} ${-track/2} ${wheel_vertical_offset}" rpy="3.14 0 0" />
+        <origin xyz="${-wheelbase/2} ${-track/2} ${wheel_vertical_offset}" rpy="1.57 0 0" />
     </xacro:scout_mini_wheel>
-    <xacro:sensor_macro parent_link="base_link">
+    <xacro:sensor_macro parent_link="base_link" sim="$(arg sim)">
         <origin xyz="0.01 0 0.07" rpy="0 0 0"/>
     </xacro:sensor_macro>
+    <!-- Additional definitions -->
+    <xacro:include filename="$(arg urdf_extras)" />
+    <!-- Gazebo definitions  -->
+    <xacro:include filename="scout_mini.gazebo" />
+    <ros2_control name="ScoutMiniSystem" type="system">
+        <hardware>
+            <plugin>gz_ros2_control/GazeboSimSystem</plugin>
+        </hardware>
+        <joint name="front_left_wheel">
+            <command_interface name="velocity"/>
+            <state_interface name="position"/>
+            <state_interface name="velocity"/>
+        </joint>
+        <joint name="front_right_wheel">
+            <command_interface name="velocity"/>
+            <state_interface name="position"/>
+            <state_interface name="velocity"/>
+        </joint>
+        <joint name="rear_left_wheel">
+            <command_interface name="velocity"/>
+            <state_interface name="position"/>
+            <state_interface name="velocity"/>
+        </joint>
+        <joint name="rear_right_wheel">
+            <command_interface name="velocity"/>
+            <state_interface name="position"/>
+            <state_interface name="velocity"/>
+        </joint>
+    </ros2_control>
 </robot>

File: ros2_ws/src/scoutmini_description/urdf/sensors.xacro (robot description, xacro)
@@ -1,12 +1,14 @@
 <?xml version="1.0"?>
 <robot xmlns:xacro="http://ros.org/wiki/xacro">
-  <xacro:macro name="sensor_macro" params="parent_link:=base_link *origin">
+  <xacro:macro name="sensor_macro" params="parent_link:=base_link sim:=false *origin">
     <xacro:arg name="camera_name"   default="zed2" />
     <xacro:arg name="camera_model"  default="zed2" />
-    <!-- ZED -->
-    <xacro:include filename="$(find zed_wrapper)/urdf/zed_macro.urdf.xacro" />
-    <xacro:zed_camera name="$(arg camera_name)" model="$(arg camera_model)" custom_baseline="0.0" enable_gnss="false">
-        <origin xyz="0 0 0" rpy="0 0 0"/>
-    </xacro:zed_camera>
+    <xacro:unless value="${sim}">
+      <!-- Real ZED camera for the physical robot. -->
+      <xacro:include filename="$(find zed_wrapper)/urdf/zed_macro.urdf.xacro" />
+      <xacro:zed_camera name="$(arg camera_name)" model="$(arg camera_model)" custom_baseline="0.0" enable_gnss="false">
+        <origin xyz="0 0 0" rpy="0 0 0"/>
+      </xacro:zed_camera>
+    </xacro:unless>
     <!-- Sensor Link -->
     <link name="sensor_link">
@@ -20,6 +22,7 @@
       </visual>
       <collision>
-        <geometry>
-          <mesh filename="file://$(find scoutmini_description)/meshes/sensors.dae" scale="1 1 1"/>
+        <origin xyz="0 0 0.06" rpy="0 0 0"/>
+        <geometry>
+          <box size="0.32 0.18 0.12"/>
         </geometry>
       </collision>
@@ -49,4 +52,13 @@
       <origin xyz="-0.075 0.0 0.12" rpy="0 0 0"/>
     </joint>
+    <gazebo reference="imu">
+      <sensor name="imu_sensor" type="imu">
+        <always_on>true</always_on>
+        <update_rate>100</update_rate>
+        <visualize>false</visualize>
+        <topic>/imu/data</topic>
+        <gz_frame_id>imu</gz_frame_id>
+      </sensor>
+    </gazebo>
     <!-- Velodyne LiDAR Link -->
     <link name="velodyne">
@@ -62,4 +74,33 @@
       <origin xyz="0.08 0.0 0.21" rpy="0 0 0"/>
     </joint>
+    <gazebo reference="velodyne">
+      <sensor name="lidar_sensor" type="gpu_lidar">
+        <always_on>true</always_on>
+        <update_rate>10</update_rate>
+        <visualize>true</visualize>
+        <topic>/scan</topic>
+        <gz_frame_id>velodyne</gz_frame_id>
+        <lidar>
+          <scan>
+            <horizontal>
+              <samples>720</samples>
+              <resolution>1</resolution>
+              <min_angle>-3.14159</min_angle>
+              <max_angle>3.14159</max_angle>
+            </horizontal>
+          </scan>
+          <range>
+            <min>0.12</min>
+            <max>20.0</max>
+            <resolution>0.01</resolution>
+          </range>
+          <noise>
+            <type>gaussian</type>
+            <mean>0.0</mean>
+            <stddev>0.01</stddev>
+          </noise>
+        </lidar>
+      </sensor>
+    </gazebo>
     <!-- Intermediate link to represent the geometry between sensor_link and cameras -->
     <link name="sensor_to_cams_link">
@@ -91,5 +132,27 @@
       <origin xyz="-0.16 0 0.0" rpy="0 0 0"/>  <!-- Adjust position -->
     </joint>
-    <!-- Add a joint to connect the ZED Camera to the robot -->
+    <xacro:if value="${sim}">
+      <!-- Simulated ZED replacement: a normal forward-facing RGB camera. -->
+      <link name="$(arg camera_name)_camera_link">
+        <visual>
+          <geometry>
+            <box size="0.09 0.16 0.05"/>
+          </geometry>
+          <material name="sim_zed_camera_material">
+            <color rgba="0.05 0.05 0.05 1.0"/>
+          </material>
+        </visual>
+        <collision>
+          <geometry>
+            <box size="0.09 0.16 0.05"/>
+          </geometry>
+        </collision>
+        <inertial>
+          <mass value="0.15"/>
+          <origin xyz="0 0 0" rpy="0 0 0"/>
+          <inertia ixx="0.0001" ixy="0" ixz="0" iyy="0.0001" iyz="0" izz="0.0001"/>
+        </inertial>
+      </link>
+    </xacro:if>
     <joint name="$(arg camera_name)_joint" type="fixed">
       <parent link="sensor_to_cams_link"/>
@@ -97,16 +160,96 @@
       <origin xyz="0.055 0.0 0.415" rpy="0 0 0"/>
     </joint>
-    <link name="360_link">
-      <inertial>
-        <mass value="0.5"/>
-        <origin xyz="0 0 0" rpy="0 0 0"/>
-        <inertia ixx="0.0003" ixy="0" ixz="0" iyy="0.0003" iyz="0" izz="0.0003"/>
-      </inertial>
-    </link>
-    <joint name="360_joint" type="fixed">
+    <xacro:if value="${sim}">
+      <link name="$(arg camera_name)_camera_optical_frame"/>
+      <joint name="$(arg camera_name)_camera_optical_joint" type="fixed">
+        <parent link="$(arg camera_name)_camera_link"/>
+        <child link="$(arg camera_name)_camera_optical_frame"/>
+        <origin xyz="0.045 0 0" rpy="-1.57079632679 0 -1.57079632679"/>
+      </joint>
+      <gazebo reference="$(arg camera_name)_camera_optical_frame">
+        <sensor name="$(arg camera_name)_rgb_camera" type="camera">
+          <always_on>true</always_on>
+          <update_rate>30</update_rate>
+          <visualize>true</visualize>
+          <topic>/$(arg camera_name)/zed_node/rgb/color/rect/image</topic>
+          <gz_frame_id>$(arg camera_name)_camera_optical_frame</gz_frame_id>
+          <camera>
+            <horizontal_fov>1.3962634</horizontal_fov>
+            <image>
+              <width>1280</width>
+              <height>720</height>
+              <format>R8G8B8</format>
+            </image>
+            <clip>
+              <near>0.05</near>
+              <far>50.0</far>
+            </clip>
+            <noise>
+              <type>gaussian</type>
+              <mean>0.0</mean>
+              <stddev>0.005</stddev>
+            </noise>
+          </camera>
+        </sensor>
+      </gazebo>
+    </xacro:if>
+    <!-- Simulated Insta360 replacement: a normal RGB camera publishing on the equirectangular image topic. -->
+    <link name="insta360_camera_link">
+      <visual>
+        <geometry>
+          <cylinder radius="0.035" length="0.08"/>
+        </geometry>
+        <material name="sim_insta360_camera_material">
+          <color rgba="0.02 0.02 0.02 1.0"/>
+        </material>
+      </visual>
+      <collision>
+        <geometry>
+          <cylinder radius="0.035" length="0.08"/>
+        </geometry>
+      </collision>
+      <inertial>
+        <mass value="0.12"/>
+        <origin xyz="0 0 0" rpy="0 0 0"/>
+        <inertia ixx="0.00008" ixy="0" ixz="0" iyy="0.00008" iyz="0" izz="0.00008"/>
+      </inertial>
+    </link>
+    <joint name="insta360_camera_joint" type="fixed">
       <parent link="sensor_to_cams_link"/>
-      <child link="360_link"/>
+      <child link="insta360_camera_link"/>
       <origin xyz="0.0 0.0 0.60" rpy="0 0 0"/>
     </joint>
+    <link name="insta360_camera_optical_frame"/>
+    <joint name="insta360_camera_optical_joint" type="fixed">
+      <parent link="insta360_camera_link"/>
+      <child link="insta360_camera_optical_frame"/>
+      <origin xyz="0.035 0 0" rpy="-1.57079632679 0 -1.57079632679"/>
+    </joint>
+    <gazebo reference="insta360_camera_optical_frame">
+      <sensor name="insta360_rgb_camera" type="camera">
+        <always_on>true</always_on>
+        <update_rate>15</update_rate>
+        <visualize>true</visualize>
+        <topic>/equirectangular/image</topic>
+        <gz_frame_id>insta360_camera_optical_frame</gz_frame_id>
+        <camera>
+          <horizontal_fov>1.57079632679</horizontal_fov>
+          <image>
+            <width>1280</width>
+            <height>720</height>
+            <format>R8G8B8</format>
+          </image>
+          <clip>
+            <near>0.05</near>
+            <far>50.0</far>
+          </clip>
+          <noise>
+            <type>gaussian</type>
+            <mean>0.0</mean>
+            <stddev>0.005</stddev>
+          </noise>
+        </camera>
+      </sensor>
+    </gazebo>
   </xacro:macro>
 </robot>
